Commit message: Add utils to create color map.

File: config/robot.urdf.xacro (robot description, xacro)
@@ -21,8 +21,8 @@
     <origin xyz="0 0 0" rpy="0 0 0" />
   </joint>
-  <link name="laser_sensor_frame"> </link>
+  <link name="rs_helios_top"> </link>
   <joint name="laser_joint" type="fixed">
     <parent link="imu_link" />
-    <child link="laser_sensor_frame" />
+    <child link="rs_helios_top" />
     <origin xyz="0 0 0" rpy="0 0 0" />
   </joint>
